File: corne-chocolate-5col/pcb/corne-chocolate.kicad_pcb (KiCad board)
At the start: 2 copper layers, 256 x 105.6 mm, 152 parts, among them J1 MJ-4PP-9, J2 OLED, J3 MJ-4PP-9, J4 OLED, SW10 SW_PUSH, SW11 SW_PUSH, SW12 SW_PUSH, SW14 SW_PUSH, SW15 SW_PUSH, SW16 SW_PUSH, SW17 SW_PUSH, SW18 SW_PUSH, SW19 SW_PUSH, SW2 SW_PUSH, SW20 SW_PUSH, SW21 SW_PUSH, SW23 SW_PUSH, SW24 SW_PUSH, SW25 SW_PUSH, SW26 SW_PUSH, SW27 SW_PUSH, SW29 SW_PUSH, SW3 SW_PUSH, SW30 SW_PUSH, SW31 SW_PUSH, SW32 SW_PUSH, SW33 SW_PUSH, SW35 SW_PUSH, SW36 SW_PUSH, SW37 SW_PUSH, SW38 SW_PUSH, SW39 SW_PUSH, SW4 SW_PUSH, SW40 SW_PUSH, SW41 SW_PUSH, SW42 SW_PUSH, SW5 SW_PUSH, SW6 SW_PUSH, SW8 SW_PUSH, SW9 SW_PUSH, U1 ProMicro, U2 ProMicro

Commit message: update corne choc v3 5col, add unrouted version for the neater people
Routing:
- net col1: track 0.00 -> 135.7 mm, vias 0 -> 11
- net col2: track 0.00 -> 124.6 mm, vias 0 -> 6
- net row0: track 0.00 -> 121.9 mm, vias 0 -> 7
- net col3: track 0.00 -> 121.8 mm, vias 0 -> 10
- net row2: track 0.00 -> 117.7 mm, vias 0 -> 6
- net row1: track 0.00 -> 113.2 mm, vias 0 -> 6
- net col4: track 0.00 -> 99.3 mm, vias 0 -> 9
- net row3: track 0.00 -> 89.9 mm, vias 0 -> 2
- net col5: track 0.00 -> 80.2 mm, vias 0 -> 10
- net GND: track 0.00 -> 63.1 mm, vias 0 -> 31
- net VCC: track 466.1 -> 514.3 mm, vias 4 -> 6
- net data: track 0.00 -> 45.4 mm, vias 0 -> 2
- net Net-(D21-Pad2): track 0.00 -> 42.4 mm, vias 0 -> 6
- net reset: track 0.00 -> 40.1 mm, vias 0 -> 4
- net SDA: track 0.00 -> 31.7 mm, vias 0 -> 1
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- added copper zone on B.Cu, net GND
- added copper zone on F.Cu, net GND
- added copper zone on B.Cu, net GNDA
- added copper zone on F.Cu, net GNDA
